File: Ruler_KiCad/Ruler_KiCad.kicad_pcb (KiCad board)
At the start: 2 copper layers, 155 x 30 mm, 24 parts

Commit message: Added V2
Other:
- board text added: "Designed by Ben Smith 2023"
- board text removed: "Designed by Ben Smith 2021"
